File: PowerSupply.kicad_sch (KiCad schematic)
At the start: 14 parts, among them J301 BATT, SW301 PWR, U301 TPS60121A, U302 TPS60121A

Commit message: LEDs and footprints
Parts:
- L301, L302: footprint (none) -> Inductor_SMD:L_Abracon_ASPI-4030S
- SW301: footprint (none) -> PCM_4ms_Switch:Switch_Toggle_SPST_SubMini
Changed lines of the file:
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@@
 			)
 		)
-		(property "Footprint" ""
+		(property "Footprint" "Inductor_SMD:L_Abracon_ASPI-4030S"
 			(at 192.278 77.724 0)
 			(effects
@@
 			)
 		)
-		(property "Footprint" ""
+		(property "Footprint" "Inductor_SMD:L_Abracon_ASPI-4030S"
 			(at 113.538 75.184 0)
 			(effects
@@
 			)
 		)
-		(property "Footprint" ""
+		(property "Footprint" "PCM_4ms_Switch:Switch_Toggle_SPST_SubMini"
 			(at 60.96 43.434 0)
 			(effects
